File: avr-module/avr-module.brd (EAGLE design)
At the start: 55.9 x 55.9 mm, 31 parts, among them U1 ATMEGA32U4-AUR

Commit message: more circuit changes
Parts:
- added C3, C4: 100 nF, rcl:C0805
- added LD1: (no value), led:DUOLED-C-5MM
- added Q1: (no value), crystal:HC49/S
- added S1, S2: (no value), switch:320-916
- added X1: 87758-0616, con-molex:87758-0616
- moved R12 42.9 mm to (49.5, 47.0), turned to 270 degrees
- moved R15 42.9 mm to (29.8, 47.0), turned to 90 degrees
- moved R17 42.9 mm to (29.8, 8.89), turned to 90 degrees
- moved R13 27.4 mm to (49.5, 27.9), turned to 270 degrees
- moved R14 27.4 mm to (49.5, 8.89), turned to 270 degrees
- moved R16 19.7 mm to (29.8, 27.9), turned to 90 degrees
Connections:
- new net N$1: R12.2, U1.41
- new net N$10: C3.1, Q1.1, U1.17
- new net N$2: R13.2, U1.40
- new net N$3: R14.2, U1.39
- new net N$4: R15.2, U1.38
- new net N$5: R16.2, U1.37
- new net N$6: R17.2, U1.36
- new net N$7: U1.3
- new net N$8: U1.4
- new net N$9: C4.1, Q1.2, U1.16
- net +3V3: now also R12.3, R13.3, R14.3, R15.3, R17.3
- net GND: now also C3.2, C4.2, R12.1, R12.4, R12.5, R13.1, R13.4, R13.5, R14.1, R14.4, R14.5, R15.1, R15.4, R15.5, R16.1, R16.4, R16.5, R17.1, R17.4, R17.5
- net SPI_MISO: now also U1.11
- net SPI_MOSI: now also U1.10
- net SPI_SCK: now also U1.9
- net VMON: now also U1.25
