File: avr-module/avr-module.sch (EAGLE design)
At the start: 31 parts, among them U1 ATMEGA32U4-AUR

Commit message: more circuit changes
Parts:
- added C3, C4: 100 nF, rcl:C-EUC0805
- added LD1: (no value), led:DUOLED-RY-C
- added Q1: (no value), crystal:CRYSTALHC49S
- added S1, S2: (no value), switch:320-916
- added X1: 87758-0616, con-molex:87758-0616
Connections:
- new net N$1: R12.2, U1.PF0_(ADC0)
- new net N$10: C3.1, Q1.1, U1.XTAL1
- new net N$2: R13.2, U1.PF1_(ADC1)
- new net N$3: R14.2, U1.PF4_(ADC4/TCK)
- new net N$4: R15.2, U1.PF5_(ADC5/TMS)
- new net N$5: R16.2, U1.PF6_(ADC6/TDO)
- new net N$6: R17.2, U1.PF7_(ADC7/TDI)
- new net N$7: U1.D-
- new net N$8: U1.D+
- new net N$9: C4.1, Q1.2, U1.XTAL2
- net +3V3: now also R12.3, R13.3, R14.3, R15.3, R17.3
- net GND: now also C3.2, C4.2, R12.1, R12.MT1, R12.MT2, R13.1, R13.MT1, R13.MT2, R14.1, R14.MT1, R14.MT2, R15.1, R15.MT1, R15.MT2, R16.1, R16.MT1, R16.MT2, R17.1, R17.MT1, R17.MT2
- net SPI_MISO: now also U1.(PDO/PCINT3/MISO)_PB3
- net SPI_MOSI: now also U1.(PDI/PCINT2/MOSI)_PB2
- net SPI_SCK: now also U1.(PCINT1/SCLK)_PB1
- net VMON: now also U1.PD4_(ICP1/ADC8
Other:
- moved on the sheet: C1, C2, D1, D11, D2, D3, D4, D5, D6, D7, D8, D9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
